File: mt_pmodsma.kicad_pcb (KiCad board)
At the start: 2 copper layers, 74.4 x 24.9 mm, 21 parts, among them J1 Conn_Coaxial, J2 Conn_Coaxial, J3 Conn_Coaxial, J4 Conn_Coaxial, J5 Conn_Coaxial, J6 Conn_Coaxial, J7 Conn_Coaxial, J8 Conn_Coaxial, J9 Conn_02x06_Odd_Even

Commit message: first gerber
Routing:
- net GND: track 380.0 -> 373.1 mm, vias 4 -> 3
- net Net-(J9-Pad1): track 24.3 -> 24.9 mm
- net Net-(J9-Pad3): track 51.3 -> 51.9 mm
- net Net-(J9-Pad2): track 29.4 -> 30.0 mm
- net Net-(J9-Pad4): track 56.4 -> 57.0 mm
